File: Esquema Elétrico/17103448.brd (EAGLE design)
At the start: 48.7 x 43.4 mm, 28 parts, among them IC1 STM32L031K6T6TR, IC3 LD117ADT-TR, IC5 LD117ADT-TR, Q1 FC-12M, U1 BMP280, X1 MINI-USB-SHIELD-UX60A-MB-5ST, X2 SPB5

Commit message: fixing drop
Parts:
- moved R3 0.51 mm to (19.3, 35.8)
- moved LED2 0.51 mm to (18.8, 32.8)
Changed lines of the file:
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@@
 <attribute name="SPICEPREFIX" value="R" x="-33.02" y="113.03" size="1.778" layer="27" rot="R180" display="off"/>
 </element>
-<element name="R3" library="rcl" library_urn="urn:adsk.eagle:library:334" package="R0805" package3d_urn="urn:adsk.eagle:package:23553/2" value="300" x="19.812" y="35.814" smashed="yes" rot="R180">
-<attribute name="NAME" x="17.907" y="36.068" size="0.8128" layer="25" rot="R180"/>
-<attribute name="POPULARITY" value="85" x="-27.178" y="99.314" size="1.778" layer="27" rot="R180" display="off"/>
-<attribute name="SPICEPREFIX" value="R" x="-27.178" y="99.314" size="1.778" layer="27" rot="R180" display="off"/>
+<element name="R3" library="rcl" library_urn="urn:adsk.eagle:library:334" package="R0805" package3d_urn="urn:adsk.eagle:package:23553/2" value="300" x="19.304" y="35.814" smashed="yes" rot="R180">
+<attribute name="NAME" x="17.399" y="36.068" size="0.8128" layer="25" rot="R180"/>
+<attribute name="POPULARITY" value="85" x="-27.686" y="99.314" size="1.778" layer="27" rot="R180" display="off"/>
+<attribute name="SPICEPREFIX" value="R" x="-27.686" y="99.314" size="1.778" layer="27" rot="R180" display="off"/>
 </element>
 <element name="U1" library="BMP280" package="XDCR_BMP280" value="BMP280" x="23.622" y="35.306" smashed="yes" rot="R90">
@@
 <element name="U$1" library="dicons" package="FIDUCIAL_G10" value="" x="40.64" y="24.384" smashed="yes"/>
 <element name="U$2" library="holes" library_urn="urn:adsk.eagle:library:237" package="3,0" package3d_urn="urn:adsk.eagle:package:14277/1" value="" x="45.72" y="18.034" smashed="yes"/>
-<element name="LED2" library="led" library_urn="urn:adsk.eagle:library:259" package="NFSG036BT" package3d_urn="urn:adsk.eagle:package:15848/1" value="NFSG036BT" x="19.304" y="32.766" smashed="yes">
-<attribute name="NAME" x="16.891" y="31.496" size="0.8128" layer="25" rot="R90"/>
-<attribute name="POPULARITY" value="0" x="19.304" y="32.766" size="1.778" layer="27" display="off"/>
+<element name="LED2" library="led" library_urn="urn:adsk.eagle:library:259" package="NFSG036BT" package3d_urn="urn:adsk.eagle:package:15848/1" value="NFSG036BT" x="18.796" y="32.766" smashed="yes">
+<attribute name="NAME" x="16.383" y="31.496" size="0.8128" layer="25" rot="R90"/>
+<attribute name="POPULARITY" value="0" x="18.796" y="32.766" size="1.778" layer="27" display="off"/>
 </element>
 <element name="U$3" library="holes" library_urn="urn:adsk.eagle:library:237" package="3,0" package3d_urn="urn:adsk.eagle:package:14277/1" value="" x="8.89" y="31.75" smashed="yes"/>
@@
 <contactref element="LED2" pad="C"/>
 <wire x1="24.597" y1="34.506" x2="23.297" y2="34.506" width="0" layer="19" extent="1-1"/>
-<wire x1="22.647" y1="36.106" x2="23.297" y2="34.506" width="0" layer="19" extent="1-1"/>
 <wire x1="11.75" y1="46.99" x2="14.92" y2="49.53" width="0" layer="19" extent="1-1"/>
 <wire x1="29.21" y1="40.32" x2="24.39" y2="38.942" width="0" layer="19" extent="1-1"/>
@@
 <contactref element="R3" pad="2"/>
 <contactref element="IC1" pad="9"/>
-<wire x1="18.862" y1="35.814" x2="18.79" y2="35.886" width="0.6096" layer="1"/>
-<wire x1="18.79" y1="35.886" x2="18.79" y2="38.942" width="0.6096" layer="1"/>
+<wire x1="18.354" y1="35.814" x2="18.79" y2="36.25" width="0.6096" layer="1"/>
+<wire x1="18.79" y1="36.25" x2="18.79" y2="38.942" width="0.6096" layer="1"/>
 </signal>
 <signal name="5V">
@@
 <contactref element="LED2" pad="A"/>
 <contactref element="R3" pad="1"/>
-<wire x1="20.762" y1="35.814" x2="20.762" y2="32.874" width="0.8128" layer="1"/>
-<wire x1="20.762" y1="32.874" x2="20.654" y2="32.766" width="0.8128" layer="1"/>
+<wire x1="20.254" y1="35.814" x2="20.254" y2="32.874" width="0.8128" layer="1"/>
+<wire x1="20.254" y1="32.874" x2="20.146" y2="32.766" width="0.8128" layer="1"/>
 </signal>
 </signals>
